File: esp32_c3_custom_board/esp32_c3_custom_board.kicad_sch (KiCad schematic)
At the start: 51 parts, among them IC1 ESP32-C3, IC2 GD25Q16CTEGR, IC3 SMD_IC_SY8089AAAC, J1 USB-C Connector, U1 ESD Protection, U2 SPX3819M5-L-3-3, Y1 830108208709_crystal

Commit message: final design yallahhh
Parts:
- added C19, C20, C21: 100nF, Capacitor_SMD:C_0603_1608Metric_Pad1.08x0.95mm_HandSolder, symbol Device:C
- added I2C1, UART1: ~, JST_Connectors:JST-PH2.0mm, symbol JST_Connectors:JST-PH2.0mm
- renumbered U1 to ESD1, IC3 to EX-Vpp1, IC2 to Flash1, U2 to USB-Vpp1, JST1 to Vpp-extern1
Connections:
- net +3.3V: now also C19.1, C20.1, C21.1
- net GND: now also C19.2, C20.2, C21.2
- net SCL: now also I2C1.2 (V-)
- net SDA: now also I2C1.1 (V+)
- net GPIO10: now reaches IC1.16 (GPIO10)
- net UART_RX: now reaches IC1.27 (U0RXD)
- net UART_RX: now also UART1.1 (V+)
- net UART_TX: now reaches IC1.28 (U0TXD)
- net UART_TX: now also UART1.2 (V-)
- net GPIO2: now reaches IC1.6 (GPIO2)
