File: esp32_c3_custom_board/esp32_c3_custom_board.kicad_pcb (KiCad board)
At the start: 2 copper layers, 44 parts, among them IC1 ESP32-C3, IC2 GD25Q16CTEGR, J1 USB-C Connector, U1 ESD Protection, U2 SPX3819M5-L-3-3, Y1 830108208709_crystal

Commit message: .
Parts:
- added C17: 22u, Capacitor_SMD:C_0201_0603Metric, F.Cu at (148.4, 133.2)
- added C18: 22u, Capacitor_SMD:C_0201_0603Metric, F.Cu at (149.3, 137.3)
- added IC3: SMD_IC_SY8089AAAC, SY8089AAAC:SOT95P285X140-5N, F.Cu at (145.7, 134.3)
- added JST1: ~, JST_Connectors:JST-PH2.0mm, F.Cu at (154.8, 134.4)
- added L3: 2.2u, Inductor_SMD:L_0201_0603Metric, F.Cu at (147.0, 137.3)
- added R16: 220k, Resistor_SMD:R_0201_0603Metric, F.Cu at (144.6, 137.3)
- added R17: 47k, Resistor_SMD:R_0201_0603Metric, F.Cu at (143.4, 133.1)
- L1, L2: footprint Inductor_SMD:L_0603_1608Metric -> Inductor_SMD:L_0201_0603Metric
- moved MonoAnt1 64.9 mm to (124.9, 151.0), turned to 180 degrees
- moved J1 63.4 mm to (153.5, 149.6), turned to 90 degrees
- moved D2 61.2 mm to (135.3, 153.7), turned to -90 degrees
- moved R9 54.8 mm to (144.6, 150.7), turned to 180 degrees
- moved C5 53.5 mm to (142.3, 154.4), turned to -90 degrees
- moved D1 52.6 mm to (145.6, 141.4), turned to 180 degrees
- moved C9 52.4 mm to (140.7, 147.9), turned to -90 degrees
- moved R10 52.1 mm to (144.6, 149.6)
- moved C10 52.0 mm to (144.3, 147.8), turned to -90 degrees
- moved L2 50.4 mm to (142.9, 147.6), turned to 180 degrees
- moved C6 50.1 mm to (142.3, 152.5), turned to 90 degrees
- moved R13 49.7 mm to (133.3, 155.0), turned to -90 degrees
- moved C11 49.5 mm to (141.6, 147.9), turned to -90 degrees
- moved R1 47.0 mm to (129.6, 145.3)
- moved R7 46.4 mm to (140.9, 152.8)
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Connections:
- C12 pad 2: unconnected-(C12-Pad2) -> GND
- IC1 pad 17: unconnected-(IC1-VDD3P3_CPU-Pad17) -> +3.3V
- IC1 pad 2: unconnected-(IC1-VDD3P3_1-Pad2) -> +3.3V
- IC1 pad 3: unconnected-(IC1-VDD3P3_2-Pad3) -> +3.3V
- IC1 pad 31: unconnected-(IC1-VDDA_1-Pad31) -> +3.3V
- IC1 pad 32: unconnected-(IC1-VDDA_2-Pad32) -> +3.3V
Routing:
- net +3.3V: track 0.00 -> 115.3 mm, vias 0 -> 5
- net Net-(IC1-GPIO18): track 0.00 -> 32.2 mm, vias 0 -> 2
- net Net-(IC1-GPIO19): track 0.00 -> 30.5 mm, vias 0 -> 2
- net /SPI_D: track 0.00 -> 20.9 mm, vias 0 -> 2
- net /VDD_SPI: track 0.00 -> 20.7 mm, vias 0 -> 2
- net Net-(IC1-CHIP_EN): track 0.00 -> 19.9 mm, vias 0 -> 2
- net /GPIO3: track 0.00 -> 18.8 mm
- net /SPI_CLK: track 0.00 -> 17.8 mm, vias 0 -> 2
- net GND: track 0.00 -> 17.7 mm, vias 0 -> 2
- net VBUS: track 0.00 -> 16.7 mm, vias 0 -> 3
- net /SCL: track 0.00 -> 16.5 mm, vias 0 -> 2
- net /SDA: track 0.00 -> 15.8 mm, vias 0 -> 2
- net /SPI_HD: track 0.00 -> 13.4 mm, vias 0 -> 2
- net Net-(IC3-EN): track 0.00 -> 12.5 mm
- net Net-(MonoAnt1-Feed): track 0.00 -> 11.9 mm
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- added copper zone on F.Cu, net GND
Other:
- board outline added: 48.1 x 25.4 mm

Commit message: .
Parts:
- C1, C13, C15, C16, C2, C5, C6: footprint Capacitor_SMD:C_0201_0603Metric -> Capacitor_SMD:C_0402_1005Metric_Pad0.74x0.62mm_HandSolder
- C10, C11, C12, C14, C3, C4, C7, C8, C9: footprint Capacitor_SMD:C_0201_0603Metric -> Capacitor_SMD:C_0603_1608Metric_Pad1.08x0.95mm_HandSolder
- C17, C18: footprint Capacitor_SMD:C_0201_0603Metric -> Capacitor_SMD:C_0805_2012Metric_Pad1.18x1.45mm_HandSolder
- L1, L2, L3: footprint Inductor_SMD:L_0201_0603Metric -> Inductor_SMD:L_0603_1608Metric_Pad1.05x0.95mm_HandSolder
- MonoAnt1: footprint Footprint_Lib:Mono_Ant -> RF_Antenna:Texas_SWRA117D_2.4GHz_Right
- R1, R10, R14, R15, R2, R3, R4, R5, R6, R7, R8, R9: footprint Resistor_SMD:R_0201_0603Metric -> Resistor_SMD:R_0402_1005Metric_Pad0.72x0.64mm_HandSolder
- R11, R12, R13, R16, R17: footprint Resistor_SMD:R_0201_0603Metric -> Resistor_SMD:R_0603_1608Metric_Pad0.98x0.95mm_HandSolder
- moved JST1 88.2 mm to (74.2, 170.2), turned to 0 degrees
- moved D1 79.3 mm to (70.3, 166.4), turned to 0 degrees
- moved IC2 78.3 mm to (58.6, 150.5)
- moved IC3 77.1 mm to (75.8, 166.8), turned to 0 degrees
- moved D2 67.1 mm to (70.3, 170.3), turned to 0 degrees
- moved C7 65.2 mm to (82.4, 134.1)
- moved C8 65.1 mm to (82.4, 136.6)
- moved HM1 62.3 mm to (70.0, 143.0)
- moved C10 62.2 mm to (82.4, 141.6), turned to 0 degrees
- moved L3 60.5 mm to (86.7, 141.6), turned to 0 degrees
- moved C9 59.0 mm to (82.4, 139.1), turned to 0 degrees
- moved C11 58.1 mm to (86.7, 129.1), turned to 0 degrees
- moved C18 57.9 mm to (92.3, 147.4)
- moved C17 57.2 mm to (92.3, 144.4), turned to 0 degrees
- moved L2 56.8 mm to (86.7, 139.1), turned to 0 degrees
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Routing:
- net +3.3V: track 115.3 -> 0.00 mm, vias 5 -> 0
- net Net-(IC1-GPIO18): track 32.2 -> 0.00 mm, vias 2 -> 0
- net Net-(IC1-GPIO19): track 30.5 -> 0.00 mm, vias 2 -> 0
- net /SPI_D: track 20.9 -> 0.00 mm, vias 2 -> 0
- net /VDD_SPI: track 20.7 -> 0.00 mm, vias 2 -> 0
- net Net-(IC1-CHIP_EN): track 19.9 -> 0.00 mm, vias 2 -> 0
- net /GPIO3: track 18.8 -> 0.00 mm
- net /SPI_CLK: track 17.8 -> 0.00 mm, vias 2 -> 0
- net GND: track 17.7 -> 0.00 mm, vias 2 -> 0
- net VBUS: track 16.7 -> 0.00 mm, vias 3 -> 0
- net /SCL: track 16.5 -> 0.00 mm, vias 2 -> 0
- net /SDA: track 15.8 -> 0.00 mm, vias 2 -> 0
- net /SPI_HD: track 13.4 -> 0.00 mm, vias 2 -> 0
- net Net-(IC3-EN): track 12.5 -> 0.00 mm
- net Net-(MonoAnt1-Feed): track 11.9 -> 0.00 mm
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- removed copper zone on F.Cu, net GND
Other:
- board size 48.1 x 25.4 mm -> 48.3 x 26 mm

Commit message: final design yallahhh
Parts:
- added C19: 100nF, Capacitor_SMD:C_0603_1608Metric_Pad1.08x0.95mm_HandSolder, F.Cu at (133.7, 142.7)
- added C20: 100nF, Capacitor_SMD:C_0603_1608Metric_Pad1.08x0.95mm_HandSolder, F.Cu at (122.2, 135.0)
- added C21: 100nF, Capacitor_SMD:C_0603_1608Metric_Pad1.08x0.95mm_HandSolder, F.Cu at (122.2, 136.5)
- added I2C1: ~, JST_Connectors:JST-PH2.0mm, F.Cu at (129.5, 147.7)
- added UART1: ~, JST_Connectors:JST-PH2.0mm, F.Cu at (146.8, 126.0)
- moved VppExt1 106.8 mm to (171.2, 125.4), turned to -90 degrees
- moved EX-Vpp1 91.3 mm to (158.7, 128.7), turned to 180 degrees
- moved D1 89.8 mm to (154.9, 136.2), turned to 90 degrees
- moved Flash1 83.2 mm to (140.8, 137.8)
- moved S1 80.4 mm to (168.6, 133.1)
- moved C10 77.9 mm to (160.2, 142.6), turned to 180 degrees
- moved C7 76.0 mm to (158.3, 137.8)
- moved C14 75.2 mm to (161.9, 132.4), turned to 90 degrees
- moved C8 74.4 mm to (155.9, 147.8), turned to 180 degrees
- moved C17 74.1 mm to (164.5, 127.5), turned to -90 degrees
- moved L3 73.7 mm to (158.6, 125.6)
- moved R9 71.7 mm to (160.0, 145.8), turned to 180 degrees
- moved R10 71.7 mm to (160.0, 144.4)
- moved R12 71.0 mm to (161.9, 136.0), turned to 90 degrees
- moved HM1 70.4 mm to (138.7, 127.6)
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- renumbered U1 to ESD1, IC3 to EX-Vpp1, IC2 to Flash1, U2 to USB-Vpp1, JST1 to VppExt1
Connections:
- IC1 pad 16: unconnected-(IC1-GPIO10-Pad16) -> /GPIO10
- IC1 pad 27: unconnected-(IC1-U0RXD-Pad27) -> /UART_RX
- IC1 pad 28: unconnected-(IC1-U0TXD-Pad28) -> /UART_TX
- IC1 pad 6: unconnected-(IC1-GPIO2-Pad6) -> /GPIO2
Routing:
- net +3.3V: track 0.00 -> 115.6 mm, vias 0 -> 4
- net Net-(IC1-CHIP_EN): track 0.00 -> 67.9 mm, vias 0 -> 2
- net /SCL: track 0.00 -> 43.6 mm, vias 0 -> 2
- net /SDA: track 0.00 -> 35.2 mm, vias 0 -> 2
- net VBUS: track 0.00 -> 27.5 mm, vias 0 -> 2
- net /USB_DN_1: track 0.00 -> 27.5 mm, vias 0 -> 2
- net Net-(IC1-SPID): track 0.00 -> 26.8 mm, vias 0 -> 2
- net /UART_TX: track 0.00 -> 26.7 mm, vias 0 -> 2
- net /USB_DP_1: track 0.00 -> 26.4 mm, vias 0 -> 2
- net /UART_RX: track 0.00 -> 23.4 mm, vias 0 -> 2
- net Net-(IC1-SPICLK): track 0.00 -> 23.1 mm, vias 0 -> 2
- net Net-(IC1-GPIO19): track 0.00 -> 22.9 mm, vias 0 -> 2
- net Net-(IC1-GPIO18): track 0.00 -> 19.2 mm, vias 0 -> 2
- net /VDD_SPI: track 0.00 -> 19.0 mm
- net Net-(IC1-SPIHD): track 0.00 -> 17.8 mm, vias 0 -> 2
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- added copper zone on B.Cu, net GND
- added copper zone on F.Cu, net GND
Other:
- board size 48.3 x 26 mm -> 61.2 x 27.4 mm
