File: altes_design/esp32_c3_custom_board/esp32_c3_custom_board.kicad_sch (KiCad schematic)
At the start: 51 parts, among them IC1 ESP32-C3, IC2 GD25Q16CTEGR, IC3 SMD_IC_SY8089AAAC, J1 USB-C Connector, U1 ESD Protection, U2 SPX3819M5-L-3-3, Y1 830108208709_crystal

Commit message: .
Parts:
- MonoAnt1: footprint RF_Antenna:Texas_SWRA117D_2.4GHz_Right -> Footprint_Lib:Mono_Ant
Changed lines of the file:
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@@
       (effects (font (size 1.27 1.27)))
     )
-    (property "Footprint" "RF_Antenna:Texas_SWRA117D_2.4GHz_Right" (at 24.13 31.75 0)
+    (property "Footprint" "Footprint_Lib:Mono_Ant" (at 24.13 31.75 0)
       (effects (font (size 1.27 1.27)) hide)
     )
